File: ECAD/sensor_board/sensor_board.kicad_sch (KiCad schematic)
At the start: 36 parts, among them J2 Conn_01x04, J4 S4B-XH-SM4-TB, Q2 Q_PMOS_GSD, Q3 Q_PMOS_GSD, Q4 2N7002, U1 TPL5111, U2 TPS22917DBV, U3 TC2030, U4 BC805M, Y1 32.768kHz

Commit message: Updated board layout
Connections:
- net BATT_DIV: now also U4.6 (P0.16); no longer U4.10 (P0.05)
- net DONE_SIGNAL: now also U4.11 (P0.14); no longer U4.12 (P0.04)
- net FLOW_SENSE: now also U4.12 (P0.04); no longer U4.6 (P0.16)
- net NDRV: now also U4.10 (P0.05); no longer U4.7 (P0.12)
- net SENSE_CTRL: now also U4.7 (P0.12); no longer U4.11 (P0.14)
Changed lines of the file:
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@@
 	(wire
 		(pts
-			(xy 135.89 167.64) (xy 123.19 167.64)
+			(xy 73.66 180.34) (xy 86.36 180.34)
 		)
 		(stroke
@@
 	(wire
 		(pts
+			(xy 124.46 177.8) (xy 123.19 177.8)
+		)
+		(stroke
+			(width 0)
+			(type default)
+		)
+	)
+	(wire
+		(pts
 			(xy 63.5 52.07) (xy 68.58 52.07)
 		)
@@
 	(wire
 		(pts
+			(xy 124.46 175.26) (xy 123.19 175.26)
+		)
+		(stroke
+			(width 0)
+			(type default)
+		)
+	)
+	(wire
+		(pts
 			(xy 71.12 124.46) (xy 71.12 110.49)
 		)
@@
 	(wire
 		(pts
+			(xy 124.46 167.64) (xy 123.19 167.64)
+		)
+		(stroke
+			(width 0)
+			(type default)
+		)
+	)
+	(wire
+		(pts
 			(xy 143.51 50.8) (xy 143.51 52.07)
 		)
@@
 	(wire
 		(pts
-			(xy 72.39 180.34) (xy 86.36 180.34)
-		)
-		(stroke
-			(width 0)
-			(type default)
-		)
-	)
-	(wire
-		(pts
 			(xy 63.5 59.69) (xy 63.5 63.5)
 		)
@@
 	(wire
 		(pts
+			(xy 124.46 170.18) (xy 123.19 170.18)
+		)
+		(stroke
+			(width 0)
+			(type default)
+		)
+	)
+	(wire
+		(pts
 			(xy 69.85 40.64) (xy 69.85 46.99)
 		)
@@
 	(wire
 		(pts
-			(xy 72.39 182.88) (xy 86.36 182.88)
-		)
-		(stroke
-			(width 0)
-			(type default)
-		)
-	)
-	(wire
-		(pts
 			(xy 124.46 26.67) (xy 121.92 26.67)
 		)
@@
 	(wire
 		(pts
+			(xy 73.66 182.88) (xy 86.36 182.88)
+		)
+		(stroke
+			(width 0)
+			(type default)
+		)
+	)
+	(wire
+		(pts
 			(xy 73.66 40.64) (xy 69.85 40.64)
 		)
@@
 	(wire
 		(pts
-			(xy 135.89 170.18) (xy 123.19 170.18)
-		)
-		(stroke
-			(width 0)
-			(type default)
-		)
-	)
-	(wire
-		(pts
 			(xy 121.92 119.38) (xy 125.73 119.38)
 		)
@@
 	(wire
 		(pts
-			(xy 123.19 177.8) (xy 135.89 177.8)
-		)
-		(stroke
-			(width 0)
-			(type default)
-		)
-	)
-	(wire
-		(pts
 			(xy 110.49 209.55) (xy 110.49 210.82)
 		)
@@
 		(pts
 			(xy 66.04 127) (xy 74.93 127)
-		)
-		(stroke
-			(width 0)
-			(type default)
-		)
-	)
-	(wire
-		(pts
-			(xy 123.19 175.26) (xy 135.89 175.26)
 		)
 		(stroke
@@
 		)
 	)
-	(label "SENSE_CTRL"
-		(at 135.89 175.26 180)
-		(fields_autoplaced yes)
-		(effects
-			(font
-				(size 1.27 1.27)
-			)
-			(justify right bottom)
-		)
-	)
 	(label "BATT_DIV"
 		(at 107.95 210.82 180)
@@
 		)
 	)
-	(label "NDRV"
-		(at 72.39 182.88 0)
+	(label "SENSE_CTRL"
+		(at 73.66 182.88 0)
+		(fields_autoplaced yes)
+		(effects
+			(font
+				(size 1.27 1.27)
+			)
+			(justify left bottom)
+		)
+	)
+	(label "Xb"
+		(at 124.46 167.64 0)
 		(fields_autoplaced yes)
 		(effects
@@
 		)
 	)
-	(label "DONE_SIGNAL"
-		(at 124.46 172.72 0)
-		(fields_autoplaced yes)
-		(effects
-			(font
-				(size 1.27 1.27)
-			)
-			(justify left bottom)
-		)
-	)
-	(label "Xa"
-		(at 135.89 170.18 180)
-		(fields_autoplaced yes)
-		(effects
-			(font
-				(size 1.27 1.27)
-			)
-			(justify right bottom)
-		)
-	)
 	(label "SENSE_CTRL"
 		(at 146.05 40.64 0)
@@
 		)
 	)
+	(label "NDRV"
+		(at 124.46 177.8 0)
+		(fields_autoplaced yes)
+		(effects
+			(font
+				(size 1.27 1.27)
+			)
+			(justify left bottom)
+		)
+	)
 	(label "FLOW_SENSE"
 		(at 36.83 127 0)
@@
 		)
 	)
-	(label "Xb"
-		(at 135.89 167.64 180)
-		(fields_autoplaced yes)
-		(effects
-			(font
-				(size 1.27 1.27)
-			)
-			(justify right bottom)
-		)
-	)
 	(label "NDRV"
 		(at 107.95 121.92 0)
@@
 	)
 	(label "FLOW_SENSE"
+		(at 124.46 172.72 0)
+		(fields_autoplaced yes)
+		(effects
+			(font
+				(size 1.27 1.27)
+			)
+			(justify left bottom)
+		)
+	)
+	(label "FLOW_SENSE"
 		(at 72.39 101.6 180)
 		(fields_autoplaced yes)
@@
 		)
 	)
+	(label "Xa"
+		(at 124.46 170.18 0)
+		(fields_autoplaced yes)
+		(effects
+			(font
+				(size 1.27 1.27)
+			)
+			(justify left bottom)
+		)
+	)
 	(label "BATT_DIV"
-		(at 135.89 177.8 180)
-		(fields_autoplaced yes)
-		(effects
-			(font
-				(size 1.27 1.27)
-			)
-			(justify right bottom)
-		)
-	)
-	(label "FLOW_SENSE"
-		(at 72.39 180.34 0)
-		(fields_autoplaced yes)
-		(effects
+		(at 73.66 180.34 0)
+		(fields_autoplaced yes)
+		(effects
+			(font
+				(size 1.27 1.27)
+			)
+			(justify left bottom)
+		)
+	)
+	(label "DONE_SIGNAL"
+		(at 124.46 175.26 0)
+		(fields_autoplaced yes)
+		(effects

Commit message: Pushing completed layout
Parts:
- JP1: value ~ -> Sold_Jump_C
- JP4: value SolderJumper_2_Open -> Sold_Jump_O
- Q2, Q3: value Q_PMOS_GSD -> PMV48XP
Other:
- note added: "Note: J2, U3, U4 excluded from BOM"
- note removed: "Notes: - J2, U3, U4 excluded from BOM"
- note removed: "TODO: - Review mounting hole sizes and update mechanical enclosure as needed - Check polarity of U1/U2"
Changed lines of the file:
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@@
 		)
 	)
-	(text "TODO:\n- Review mounting hole sizes and update mechanical enclosure as needed\n- Check polarity of U1/U2"
+	(text "Note: J2, U3, U4 excluded from BOM"
 		(exclude_from_sim no)
-		(at 17.272 246.126 0)
+		(at 17.526 238.506 0)
 		(effects
 			(font
-				(size 1.27 1.27)
-				(thickness 0.254)
-				(bold yes)
-				(color 255 15 6 1)
-			)
-			(justify left)
-		)
-	)
-	(text "Notes:\n- J2, U3, U4 excluded from BOM"
-		(exclude_from_sim no)
-		(at 18.034 261.366 0)
-		(effects
-			(font
-				(size 1.27 1.27)
+				(size 2.54 2.54)
 				(thickness 0.254)
 				(bold yes)
@@
 			)
 		)
-		(property "Value" "Q_PMOS_GSD"
+		(property "Value" "PMV48XP"
 			(at 96.52 48.2346 90)
 			(effects
@@
 			)
 		)
-		(property "Datasheet" "~"
+		(property "Datasheet" "https://wmsc.lcsc.com/wmsc/upload/file/pdf/v2/lcsc/2201211530_TECH-PUBLIC-PMV48XP_C2959854.pdf"
 			(at 96.52 54.61 0)
 			(effects
@@
 			)
 		)
-		(property "Value" "SolderJumper_2_Open"
+		(property "Value" "Sold_Jump_O"
 			(at 96.52 39.0144 0)
 			(effects
@@
 		(on_board yes)
 		(dnp no)
-		(fields_autoplaced yes)
 		(property "Reference" "JP1"
 			(at 74.93 49.53 0)
@@
 			)
 		)
-		(property "Value" "~"
-			(at 74.93 49.53 0)
+		(property "Value" "Sold_Jump_C"
+			(at 74.93 54.864 0)
 			(effects
 				(font
@@
 			)
 		)
-		(property "Value" "Q_PMOS_GSD"
+		(property "Value" "PMV48XP"
 			(at 118.0846 34.29 90)
 			(effects
@@
 			)
 		)
-		(property "Datasheet" "~"
+		(property "Datasheet" "https://wmsc.lcsc.com/wmsc/upload/file/pdf/v2/lcsc/2201211530_TECH-PUBLIC-PMV48XP_C2959854.pdf"
 			(at 124.46 34.29 0)
 			(effects
